File: ruuviharvester_reva1/ruuviharvester_reva1.sch (KiCad schematic (older format))
At the start: 30 parts, among them P1 PIEZO, SW1 DIP_SWITCH_3POS, U1 SPV1050, U2 TS3310, U3 SOLAR_CELL

Commit message: Small mods
Parts:
- added C?: SUPER_CAP, symbol CP
Connections:
- net GND: now also U1.13 (CONF), C?.2; no longer C1.2, U1.19 (L_HV), U1.20 (IN_HV), U1.5 (LDO1_EN)
- net at C3.2, D2.1 (K), U3.1 (+): now also U1.20 (IN_HV); no longer L1.1, U1.13 (CONF)
- net +1V8: now reaches U1.11 (LDO1)
- new net: C1.2, C?.1
- new net: L1.1, U1.19 (L_HV)
- new net 1V8_LDO_EN: U1.5 (LDO1_EN)
- no-connect marks 5 -> 4
Other:
- note added: "A few of the possible combinations:\n\n* 1-3 cell solar panel and SPV1050 in boost mode\n* 6-18 cell solar panel and SPV1050 in buck-boost mode\n* Piezo element(s) and SPV1050 in boost mode\n* TEG element and SPV1050 in boost mode\n* Wideband antenna for RF energy scavenging and SPV1050 in boost mode\n\n+\n\n* Cap-XX Thinline and TS3310 @ 3V\n* Cap-XX Thinline + SPV1050 1.8V LDO\n* 2x Cap-XX Thin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"
- note added: "Boost configuration:\nCONF -> Source\nBuck-boost configuration:\nCONF -> GND"
- note added: "Boost configuration:\nIN_LV -> Inductor -> Source\nIN_HV -> GND\nL_HV -> GND\n\nBuck-boost configuration:\nIN_LV -> Inductor -> L_HV\nIN_HV -> Source\nMPP -> R1 -> IN_HV"
- note added: "If SPV1050 is configured to perform in buck-boost mode it's\nrecommended to use at least 6 cell solar panel. Otherwise might\nhappen that minumum startup voltage isn't reached in low light conditions."
- note added: "Once the harvested source is connected, the SPV1050 will\nstart boosting the voltage on the STORE pin. In the range of\n0 VSTORE < 2.6 V the voltage boost is carried on by an integrated\nhigh-efficiency charge pump, while the DC-DC converter stage\nwill remain OFF. \n"
- note removed: "Once the harvested source is connected, the SPV1050 device will\nstart boosting the voltage on the STORE pin. In the range of\n0 VSTORE < 2.6 V the voltage boost is carried on by an integrated\nhigh-efficiency charge pump, while the DC-DC converter stage\nwill remain OFF. \n"
- moved on the sheet: C1, C10, C2, C3, C4, C5, C6, C7, C8, C9, D1, D2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
